File: Board_Files/adp2384.kicad_pcb (KiCad board)
At the start: 2 copper layers, 35 x 40 mm, 26 parts, among them J1 Conn_01x02, J2 Conn_01x03, J3 Conn_01x02, U1 ADP2384

Commit message: Update A1 Release files
1. Added design information in Schematics.
2. BOM generated.
3. Updated the library path to align with the current folder structure.
4. Added 3D board file images.
5. Updated README.
Changed lines of the file:
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@@
 			(layer "F.Fab")
 		)
+		(fp_text user "*"
+			(at -3.1374 -1.25 0)
+			(layer "F.SilkS")
+			(effects
+				(font
+					(size 1 1)
+					(thickness 0.15)
+				)
+			)
+		)
+		(fp_text user "*"
+			(at -3.1374 -1.25 0)
+			(unlocked yes)
+			(layer "F.SilkS")
+			(effects
+				(font
+					(size 1 1)
+					(thickness 0.15)
+				)
+			)
+		)
+		(fp_text user "*"
+			(at -0.7626 -1.25 0)
+			(unlocked yes)
+			(layer "F.Fab")
+			(effects
+				(font
+					(size 1 1)
+					(thickness 0.15)
+				)
+			)
+		)
+		(fp_text user "*"
+			(at -0.7626 -1.25 0)
+			(layer "F.Fab")
+			(effects
+				(font
+					(size 1 1)
+					(thickness 0.15)
+				)
+			)
+		)
 		(fp_text user "${REFERENCE}"
 			(at 0 0 0)
@@
 		)
 		(embedded_fonts no)
-		(model "${KIPRJMOD}/ul_ADP2384ACPZN-R7/CP_24_12_ADI.step"
+		(model "${KIPRJMOD}/PartLibrary/ul_ADP2384ACPZN-R7/CP_24_12_ADI.step"
 			(offset
 				(xyz 0 0 0)
@@
 		)
 		(embedded_fonts no)
-		(model "${KIPRJMOD}/IHLP4040DZER3R3M01/IND_IHLP-4040DZ_VIS.step"
+		(model "${KIPRJMOD}/PartLibrary/IHLP4040DZER3R3M01/IND_IHLP-4040DZ_VIS.step"
 			(offset
 				(xyz 0 0 0)
