File: Board_Files/adp2384.kicad_sch (KiCad schematic)
At the start: 26 parts, among them J1 Conn_01x02, J2 Conn_01x03, J3 Conn_01x02, U1 ADP2384

Commit message: Update A1 Release files
1. Added design information in Schematics.
2. BOM generated.
3. Updated the library path to align with the current folder structure.
4. Added 3D board file images.
5. Updated README.
Parts:
- C4: Mfg Part No CC0603KRX7R7BB104 -> CC0603KRX7R9BB104
Other:
- note added: "ADP2384 Board"
- note added: "Connect a jumper between J2.1 and J2.2 to enable the converter"
- note added: "Input Voltage: 12V"
- note added: "Output Voltage: 3.3V Output Current: 4A Switching Frequency: 600KHz Output Ripple: 2% (66mV) Soft Start: 4ms"
- company: (none) -> ARD
- title: (none) -> ADB2384 EVL
